File: PIC14K50 USB Breakout PCB/PIC18F14K50 USB.brd (EAGLE design)
At the start: 23.8 x 40.4 mm, 33 parts, among them IC1 MAX3232EUE

Commit message: silk fix
Parts:
- moved R9 0.21 mm to (14.3, 21.0)
Routing:
- net GND: track 43.9 -> 44.6 mm
